File: beefy_linear_mosfet.kicad_pcb (KiCad board)
At the start: 4 copper layers, 70 x 100 mm, 60 parts, among them IC1 LT3090EMSE#PBF, IC2 LT3080EMS8E#PBF, J1 Conn_Coaxial, J2 MOSFET GS, J3 SupplyP, J4 SupplyN, J5 GND, J6 Conn_Coaxial, J7 Conn_Coaxial, J8 Conn_Coaxial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

Commit message: Update prototype effor so far
Parts:
- removed J5: GND, TerminalBlock:TerminalBlock_bornier-2_P5.08mm
- removed R14: 5, Resistor_THT:R_Axial_DIN0309_L9.0mm_D3.2mm_P12.70mm_Horizontal
- removed U2: TL431DBZ, Package_TO_SOT_SMD:SOT-23
- added D1: D, Diode_THT:D_DO-35_SOD27_P7.62mm_Horizontal, F.Cu at (55.0, 75.5)
- added D2: D, Diode_THT:D_DO-35_SOD27_P7.62mm_Horizontal, F.Cu at (35.2, 75.5)
- added D3: D_Zener 3.3V, Diode_THT:D_DO-35_SOD27_P7.62mm_Horizontal, F.Cu at (31.0, 61.5)
- added D4: D_Zener 15V, Diode_THT:D_DO-35_SOD27_P7.62mm_Horizontal, F.Cu at (68.5, 42.8)
- added D5: D_Zener 15V, Diode_THT:D_DO-35_SOD27_P7.62mm_Horizontal, F.Cu at (65.8, 43.5)
- C15, C5: value 220u -> A768KE107M1VLAS036; footprint Capacitor_THT:CP_Radial_D10.0mm_P5.00mm -> Capacitor_SMD:CP_Elec_8x6.7
- C18, C6: value 220u -> A768KE826M1GLAS038; footprint Capacitor_THT:CP_Radial_D10.0mm_P5.00mm -> Capacitor_SMD:CP_Elec_8x6.7
- C4: value 1n -> 10n
- R12: value 5 -> 200k; footprint Resistor_THT:R_Axial_DIN0309_L9.0mm_D3.2mm_P12.70mm_Horizontal -> SamacSys_Parts:R_1206_0805_dual
- R13: value 1000 -> 2700; footprint Resistor_THT:R_Axial_DIN0309_L9.0mm_D3.2mm_P12.70mm_Horizontal -> Resistor_THT:R_Axial_DIN0617_L17.0mm_D6.0mm_P25.40mm_Horizontal
- R2: value 250 -> 560
- R7: value 10k -> 200k; footprint Resistor_THT:R_Axial_DIN0309_L9.0mm_D3.2mm_P12.70mm_Horizontal -> SamacSys_Parts:R_1206_0805_dual
- moved R7 54.4 mm to (62.5, 29.5)
- moved R12 38.9 mm to (27.8, 35.2), turned to 270 degrees
- moved R2 8.00 mm to (39.8, 47.8)
- moved C6 3.26 mm to (61.2, 95.8)
- moved R1 3.09 mm to (28.8, 39.0)
- moved C5 3.05 mm to (29.2, 95.5)
- moved C18 3.04 mm to (51.8, 83.5)
- moved C15 2.25 mm to (40.0, 83.5)
- moved C4 2.24 mm to (28.0, 65.2)
- moved R13 2.24 mm to (67.8, 48.5)
- moved J9 1.65 mm to (51.5, 30.5)
- moved JP1 1.27 mm to (33.0, 42.8)
- moved J1 1.00 mm to (19.8, 39.5)
- moved J8 1.00 mm to (19.8, 39.5)
- moved R15 0.74 mm to (56.8, 32.2)
Connections:
- C3 pad 1: Net-(C3-Pad1) -> /Gate
- IC2 pad 9: GND -> VDDA
- J2 pad 1: Net-(C3-Pad1) -> /Gate
- J2 pad 2: Net-(C3-Pad1) -> /Gate
- J2 pad 3: Net-(C3-Pad1) -> GND
- J2 pad 4: Net-(J2-Pad4) -> /Drain
- J2 pad 5: Net-(J2-Pad4) -> GND
- Q1 pad 2: Net-(J2-Pad4) -> /Drain
- Q2 pad 2: Net-(J2-Pad4) -> /Drain
- R10 pad 1: Net-(C3-Pad1) -> /Gate
- R11 pad 1: Net-(C3-Pad1) -> /Gate
- R12 pad 1: Net-(C3-Pad1) -> GND
- R12 pad 2: Net-(C1-Pad1) -> Net-(J1-Pad1)
- R13 pad 1: Net-(J2-Pad4) -> /Drain
- R16 pad 1: Net-(J2-Pad4) -> /Drain
- R17 pad 1: Net-(J2-Pad4) -> /Drain
- R7 pad 1: GND -> Net-(C3-Pad2)
- R7 pad 2: Net-(C4-Pad1) -> /Gate
Routing:
- net Net-(C3-Pad1): track 49.5 -> 0.00 mm
- net /Gate: track 0.00 -> 30.1 mm
- net Net-(Q1-Pad3): track 33.1 -> 19.4 mm
- net VDDA: track 6.96 -> 19.5 mm, vias 8 -> 9
- net /Drain: track 0.00 -> 11.7 mm
- net Net-(R13-Pad2): track 28.7 -> 22.6 mm
- net Net-(C4-Pad1): track 34.4 -> 28.4 mm
- net VSSA: track 52.4 -> 58.4 mm
- net Net-(C1-Pad1): track 28.7 -> 24.7 mm
- net Net-(C3-Pad2): track 8.84 -> 5.71 mm
- net Net-(D4-Pad1): track 0.00 -> 3.06 mm
- net Net-(JP2-Pad1): track 4.86 -> 6.43 mm
- net Net-(C4-Pad2): track 18.9 -> 17.4 mm
- net Net-(JP1-Pad2): track 5.88 -> 6.41 mm
- net Net-(J1-Pad1): track 14.0 -> 14.5 mm
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- added copper zone on F.Cu, net /Drain
- removed copper zone on F.Cu, net Net-(J2-Pad4)
