File: beefy_linear_mosfet.sch (KiCad schematic (older format))
At the start: 60 parts, among them IC1 LT3090EMSE#PBF, IC2 LT3080EMS8E#PBF, J1 Conn_Coaxial, J2 MOSFET GS, J3 SupplyP, J4 SupplyN, J5 GND, J6 Conn_Coaxial, J7 Conn_Coaxial, J8 Conn_Coaxial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

Commit message: Update prototype effor so far
Parts:
- removed J5: GND, TerminalBlock:TerminalBlock_bornier-2_P5.08mm, symbol Connector:Screw_Terminal_01x02
- removed R14: 5, Resistor_THT:R_Axial_DIN0309_L9.0mm_D3.2mm_P12.70mm_Horizontal, symbol Device:R
- removed U2: TL431DBZ, Package_TO_SOT_SMD:SOT-23, symbol Reference_Voltage:TL431DBZ
- added D1, D2: D, Diode_THT:D_DO-35_SOD27_P7.62mm_Horizontal, symbol Device:D
- added D3: D_Zener 3.3V, Diode_THT:D_DO-35_SOD27_P7.62mm_Horizontal, symbol Device:D_Zener
- added D4, D5: D_Zener 15V, Diode_THT:D_DO-35_SOD27_P7.62mm_Horizontal, symbol Device:D_Zener
- C15, C5: value 220u -> A768KE107M1VLAS036; footprint Capacitor_THT:CP_Radial_D10.0mm_P5.00mm -> Capacitor_SMD:CP_Elec_8x6.7
- C18, C6: value 220u -> A768KE826M1GLAS038; footprint Capacitor_THT:CP_Radial_D10.0mm_P5.00mm -> Capacitor_SMD:CP_Elec_8x6.7
- C4: value 1n -> 10n
- IC1: footprint SOP65P490X110-13N -> SamacSys_Parts:SOP65P490X110-13N
- IC2: footprint SOP65P490X110-9N -> SamacSys_Parts:SOP65P490X110-9N
- R12: value 5 -> 200k; footprint Resistor_THT:R_Axial_DIN0309_L9.0mm_D3.2mm_P12.70mm_Horizontal -> SamacSys_Parts:R_1206_0805_dual
- R13: value 1000 -> 2700; footprint Resistor_THT:R_Axial_DIN0309_L9.0mm_D3.2mm_P12.70mm_Horizontal -> Resistor_THT:R_Axial_DIN0617_L17.0mm_D6.0mm_P25.40mm_Horizontal
- R2: value 250 -> 560
- R7: value 10k -> 200k; footprint Resistor_THT:R_Axial_DIN0309_L9.0mm_D3.2mm_P12.70mm_Horizontal -> SamacSys_Parts:R_1206_0805_dual
Connections:
- net GND: now also J2.3 (Pin_3), J2.5 (Pin_5), R12.1, D1.2 (A), D2.1 (K); no longer IC2.9 (EP), R7.1
- net VDDA: now also IC2.9 (EP), D1.1 (K)
- net VSSA: now also D2.2 (A)
- net at C4.1, Q1.1 (B), Q2.1 (B)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: now also D3.1 (K); no longer R7.2
- net at C4.2, JP3.2 (C), R8.2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: now also D3.2 (A)
- net Gate: now reaches C3.1, J2.1 (Pin_1), J2.2 (Pin_2), R10.1, R11.1
- net Gate: now also R7.2, D4.2 (A); no longer J2.3 (Pin_3), R12.1
- net at C1.1, C2.1, R10.2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: no longer R12.2
- net Drain: now reaches J2.4 (Pin_4), Q1.2 (C), Q2.2 (C), R13.1, R16.1, R17.1
- net Drain: now also D5.2 (A); no longer J2.5 (Pin_5)
- net at J1.1 (In), J8.1 (In), JP1.3 (B)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: now also R12.2
- net at C3.2, R15.2: now also R7.1
- new net: D4.1 (K), D5.1 (K)
Other:
- moved on the sheet: C21, C22, C3, R13, R15, R8, R9
